File: example-dev/usb-dam.kicad_sch (KiCad schematic)
At the start: 44 parts, among them J2 Conn_01x08_Pin, J3 USB_C_Receptacle, U1 MCP6002-xMC, U2 SiP32431DR3, U3 TMUX1574RSVR, U4 74LVC1G08

Commit message: layout example board
Parts:
- removed TP7, TP9 (x4): TestPoint, tuna-f1sh/jbr-kicad/Misc.pretty:TestPoint_Pad_D1.0mm_Tight, symbol Connector:TestPoint_Small
Changed lines of the file:
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@@
   (junction (at 307.848 59.944) (diameter 0) (color 0 0 0 0)
   )
-  (junction (at 273.05 200.152) (diameter 0) (color 0 0 0 0)
-  )
   (junction (at 225.806 52.07) (diameter 0) (color 0 0 0 0)
   )
@@
   (junction (at 112.268 96.774) (diameter 0) (color 0 0 0 0)
   )
-  (junction (at 273.05 202.692) (diameter 0) (color 0 0 0 0)
-  )
   (junction (at 62.484 35.814) (diameter 0) (color 0 0 0 0)
   )
   (junction (at 112.268 94.234) (diameter 0) (color 0 0 0 0)
   )
-  (junction (at 273.05 197.612) (diameter 0) (color 0 0 0 0)
-  )
   (junction (at 255.524 90.424) (diameter 0) (color 0 0 0 0)
   )
@@
   (junction (at 92.456 105.918) (diameter 0) (color 0 0 0 0)
   )
-  (junction (at 273.05 205.232) (diameter 0) (color 0 0 0 0)
-  )
   (junction (at 187.198 136.144) (diameter 0) (color 0 0 0 0)
   )
@@
   (junction (at 70.104 47.244) (diameter 0) (color 0 0 0 0)
   )
-  (junction (at 73.152 145.034) (diameter 0) (color 0 0 0 0)
-  )
   (junction (at 165.862 124.714) (diameter 0) (color 0 0 0 0)
   )
@@
   (no_connect (at 240.284 200.152))
   (no_connect (at 240.284 205.232))
-  (wire (pts (xy 280.416 202.692) (xy 273.05 202.692))
-    (stroke (width 0) (type default))
-  )
   (wire (pts (xy 49.784 187.96) (xy 49.784 179.07))
     (stroke (width 0) (type default))
@@
     (stroke (width 0) (type default))
   )
-  (wire (pts (xy 270.764 202.692) (xy 273.05 202.692))
+  (wire (pts (xy 270.764 202.692) (xy 280.416 202.692))
     (stroke (width 0) (type default))
   )
@@
     (stroke (width 0) (type default))
   )
-  (wire (pts (xy 69.85 145.034) (xy 73.152 145.034))
+  (wire (pts (xy 69.85 145.034) (xy 110.236 145.034))
     (stroke (width 0) (type default))
   )
-  (wire (pts (xy 273.05 200.152) (xy 280.416 200.152))
+  (wire (pts (xy 270.764 200.152) (xy 280.416 200.152))
     (stroke (width 0) (type default))
   )
@@
     (stroke (width 0) (type default))
   )
-  (wire (pts (xy 73.152 145.034) (xy 110.236 145.034))
-    (stroke (width 0) (type default))
-  )
   (wire (pts (xy 54.864 54.864) (xy 54.864 78.994))
     (stroke (width 0) (type default))
@@
     (stroke (width 0) (type default))
   )
-  (wire (pts (xy 280.416 205.232) (xy 273.05 205.232))
+  (wire (pts (xy 270.764 205.232) (xy 280.416 205.232))
     (stroke (width 0) (type default))
   )
@@
     (stroke (width 0) (type default))
   )
-  (wire (pts (xy 270.764 200.152) (xy 273.05 200.152))
-    (stroke (width 0) (type default))
-  )
-  (wire (pts (xy 270.764 197.612) (xy 273.05 197.612))
+  (wire (pts (xy 270.764 197.612) (xy 280.416 197.612))
     (stroke (width 0) (type default))
   )
@@
     (stroke (width 0) (type default))
   )
-  (wire (pts (xy 273.05 197.612) (xy 280.416 197.612))
-    (stroke (width 0) (type default))
-  )
   (wire (pts (xy 62.484 35.814) (xy 54.864 35.814))
     (stroke (width 0) (type default))
   )
-  (wire (pts (xy 270.764 205.232) (xy 273.05 205.232))
-    (stroke (width 0) (type default))
-  )
   (wire (pts (xy 67.564 96.774) (xy 92.456 96.774))
     (stroke (width 0) (type default))
@@
     )
   )
-  (symbol (lib_id "Connector:TestPoint_Small") (at 73.152 145.034 0) (unit 1)
-    (in_bom yes) (on_board yes) (dnp no)
-    (property "Reference" "TP7" (at 73.152 143.764 0)
-      (effects (font (size 1.27 1.27)) (justify left))
-    )
-    (property "Value" "TestPoint" (at 74.6252 144.2974 0)
-      (effects (font (size 1.27 1.27)) (justify left) hide)
-    )
-    (property "Footprint" "tuna-f1sh/jbr-kicad/Misc.pretty:TestPoint_Pad_D1.0mm_Tight" (at 78.232 145.034 0)
-      (effects (font (size 1.27 1.27)) hide)
-    )
-    (property "Datasheet" "~" (at 78.232 145.034 0)
-      (effects (font (size 1.27 1.27)) hide)
-    )
-    (property "Config" "nofit" (at 73.152 145.034 0)
-      (effects (font (size 1.27 1.27)) hide)
-    )
-    (pin "1")
-    (instances
-      (project "USB"
-        (path "/abe08c89-73f7-4625-b1e5-d5b33729a7ca"
-          (reference "TP7") (unit 1)
-        )
-      )
-      (project "spirit_logger_hardware"
-        (path "/e63e39d7-6ac0-4ffd-8aa3-1841a4541b55/cec0ac2b-8788-4205-bc11-fcadefc26e0e"
-          (reference "TP7") (unit 1)
-        )
-      )
-      (project "usb-dam"
-        (path "/eb1f9132-3dcd-4de4-9f05-c2db01d52e0f"
-          (reference "TP1") (unit 1)
-        )
-      )
-    )
-  )
   (symbol (lib_id "power:GND") (at 65.024 191.77 0) (unit 1)
     (in_bom yes) (on_board yes) (dnp no)
@@
     )
   )
-  (symbol (lib_id "Connector:TestPoint_Small") (at 273.05 197.612 0) (unit 1)
-    (in_bom yes) (on_board yes) (dnp no)
-    (property "Reference" "TP9" (at 273.05 196.215 0)
-      (effects (font (size 1.27 1.27)) (justify left))
-    )
-    (property "Value" "TestPoint" (at 274.5232 196.8754 0)
-      (effects (font (size 1.27 1.27)) (justify left) hide)
-    )
-    (property "Footprint" "tuna-f1sh/jbr-kicad/Misc.pretty:TestPoint_Pad_D1.0mm_Tight" (at 278.13 197.612 0)
-      (effects (font (size 1.27 1.27)) hide)
-    )
-    (property "Datasheet" "~" (at 278.13 197.612 0)
-      (effects (font (size 1.27 1.27)) hide)
-    )
-    (property "Config" "nofit" (at 273.05 197.612 0)
-      (effects (font (size 1.27 1.27)) hide)
-    )
-    (pin "1")
-    (instances
-      (project "USB"
-        (path "/abe08c89-73f7-4625-b1e5-d5b33729a7ca"
-          (reference "TP9") (unit 1)
-        )
-      )
-      (project "spirit_logger_hardware"
-        (path "/e63e39d7-6ac0-4ffd-8aa3-1841a4541b55/cec0ac2b-8788-4205-bc11-fcadefc26e0e"
-          (reference "TP9") (unit 1)
-        )
-      )
-      (project "usb-dam"
-        (path "/eb1f9132-3dcd-4de4-9f05-c2db01d52e0f"
-          (reference "TP10") (unit 1)
-        )
-      )
-    )
-  )
   (symbol (lib_id "Device:R_Small") (at 101.6 96.774 90) (mirror x) (unit 1)
     (in_bom yes) (on_board yes) (dnp no)
@@
     )
   )
-  (symbol (lib_id "Connector:TestPoint_Small") (at 273.05 202.692 0) (unit 1)
-    (in_bom yes) (on_board yes) (dnp no)
-    (property "Reference" "TP9" (at 273.05 201.295 0)
-      (effects (font (size 1.27 1.27)) (justify left))
-    )
-    (property "Value" "TestPoint" (at 274.5232 201.9554 0)
-      (effects (font (size 1.27 1.27)) (justify left) hide)
-    )
-    (property "Footprint" "tuna-f1sh/jbr-kicad/Misc.pretty:TestPoint_Pad_D1.0mm_Tight" (at 278.13 202.692 0)
-      (effects (font (size 1.27 1.27)) hide)
-    )
-    (property "Datasheet" "~" (at 278.13 202.692 0)
-      (effects (font (size 1.27 1.27)) hide)
-    )
-    (property "Config" "nofit" (at 273.05 202.692 0)
-      (effects (font (size 1.27 1.27)) hide)
-    )
-    (pin "1")
-    (instances
-      (project "USB"
-        (path "/abe08c89-73f7-4625-b1e5-d5b33729a7ca"
-          (reference "TP9") (unit 1)
-        )
-      )
-      (project "spirit_logger_hardware"
-        (path "/e63e39d7-6ac0-4ffd-8aa3-1841a4541b55/cec0ac2b-8788-4205-bc11-fcadefc26e0e"
-          (reference "TP9") (unit 1)
-        )
-      )
-      (project "usb-dam"
-        (path "/eb1f9132-3dcd-4de4-9f05-c2db01d52e0f"
-          (reference "TP6") (unit 1)
-        )
-      )
-    )
-  )
   (symbol (lib_id "Power_Management:SiP32431DR3") (at 177.292 138.684 0) (unit 1)
     (in_bom yes) (on_board yes) (dnp no) (fields_autoplaced)
@@
     )
   )
-  (symbol (lib_id "Connector:TestPoint_Small") (at 273.05 200.152 0) (unit 1)
-    (in_bom yes) (on_board yes) (dnp no)
-    (property "Reference" "TP9" (at 273.05 198.755 0)
-      (effects (font (size 1.27 1.27)) (justify left))
-    )
-    (property "Value" "TestPoint" (at 274.5232 199.4154 0)
-      (effects (font (size 1.27 1.27)) (justify left) hide)
-    )
-    (property "Footprint" "tuna-f1sh/jbr-kicad/Misc.pretty:TestPoint_Pad_D1.0mm_Tight" (at 278.13 200.152 0)
-      (effects (font (size 1.27 1.27)) hide)
-    )
-    (property "Datasheet" "~" (at 278.13 200.152 0)
-      (effects (font (size 1.27 1.27)) hide)
-    )
-    (property "Config" "nofit" (at 273.05 200.152 0)
-      (effects (font (size 1.27 1.27)) hide)
-    )
-    (pin "1")
-    (instances
-      (project "USB"
-        (path "/abe08c89-73f7-4625-b1e5-d5b33729a7ca"
-          (reference "TP9") (unit 1)
-        )
-      )
-      (project "spirit_logger_hardware"
-        (path "/e63e39d7-6ac0-4ffd-8aa3-1841a4541b55/cec0ac2b-8788-4205-bc11-fcadefc26e0e"
-          (reference "TP9") (unit 1)
-        )
-      )
-      (project "usb-dam"
-        (path "/eb1f9132-3dcd-4de4-9f05-c2db01d52e0f"
-          (reference "TP9") (unit 1)
-        )
-      )
-    )
-  )
   (symbol (lib_id "power:GND") (at 177.292 147.828 0) (unit 1)
     (in_bom yes) (on_board yes) (dnp no) (fields_autoplaced)
@@
         )
       )
-    )
-  )
-  (symbol (lib_id "Connector:TestPoint_Small") (at 273.05 205.232 0) (unit 1)
-    (in_bom yes) (on_board yes) (dnp no)
-    (property "Reference" "TP9" (at 273.05 203.835 0)
-      (effects (font (size 1.27 1.27)) (justify left))
-    )
-    (property "Value" "TestPoint" (at 274.5232 204.4954 0)
-      (effects (font (size 1.27 1.27)) (justify left) hide)
-    )
-    (property "Footprint" "tuna-f1sh/jbr-kicad/Misc.pretty:TestPoint_Pad_D1.0mm_Tight" (at 278.13 205.232 0)
-      (effects (font (size 1.27 1.27)) hide)
-    )
-    (property "Datasheet" "~" (at 278.13 205.232 0)
-      (effects (font (size 1.27 1.27)) hide)
-    )
-    (property "Config" "nofit" (at 273.05 205.232 0)
-      (effects (font (size 1.27 1.27)) hide)
-    )
-    (pin "1")
-    (instances
-      (project "USB"
-        (path "/abe08c89-73f7-4625-b1e5-d5b33729a7ca"
-          (reference "TP9") (unit 1)
-        )
-      )
-      (project "spirit_logger_hardware"
-        (path "/e63e39d7-6ac0-4ffd-8aa3-1841a4541b55/cec0ac2b-8788-4205-bc11-fcadefc26e0e"
-          (reference "TP9") (unit 1)
-        )
-      )
-      (project "usb-dam"
-        (path "/eb1f9132-3dcd-4de4-9f05-c2db01d52e0f"
-          (reference "TP11") (unit 1)
-        )
-      )

Commit message: example board for production
Parts:
- added TP9 (x2): TestPoint, TestPoint:TestPoint_Pad_D2.0mm, symbol Connector:TestPoint_Small
Connections:
- net USB_D+: now also TP9.1
- net USB_D-: now also TP9.1
- net DAM_RX+ renamed SWDO/TXD
- net DAM_RX- renamed ~{NRST}/RXD
Changed lines of the file:
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@@
   (junction (at 62.484 35.814) (diameter 0) (color 0 0 0 0)
   )
+  (junction (at 138.176 52.324) (diameter 0) (color 0 0 0 0)
+  )
   (junction (at 112.268 94.234) (diameter 0) (color 0 0 0 0)
   )
@@
   (junction (at 92.456 105.918) (diameter 0) (color 0 0 0 0)
   )
+  (junction (at 101.6 52.324) (diameter 0) (color 0 0 0 0)
+  )
   (junction (at 187.198 136.144) (diameter 0) (color 0 0 0 0)
   )
@@
     (stroke (width 0) (type default))
   )
+  (wire (pts (xy 133.096 52.324) (xy 138.176 52.324))
+    (stroke (width 0) (type default))
+  )
   (wire (pts (xy 371.856 112.014) (xy 371.856 122.174))
     (stroke (width 0) (type default))
@@
     (stroke (width 0) (type default))
   )
-  (wire (pts (xy 106.172 52.324) (xy 107.696 52.324))
+  (wire (pts (xy 98.552 52.324) (xy 101.6 52.324))
     (stroke (width 0) (type default))
   )
@@
     (stroke (width 0) (type default))
   )
-  (wire (pts (xy 133.096 52.324) (xy 134.366 52.324))
-    (stroke (width 0) (type default))
-  )
   (wire (pts (xy 67.564 94.234) (xy 87.122 94.234))
     (stroke (width 0) (type default))
@@
     (stroke (width 0) (type default))
   )
+  (wire (pts (xy 101.6 52.324) (xy 107.696 52.324))
+    (stroke (width 0) (type default))
+  )
   (wire (pts (xy 120.396 65.024) (xy 120.396 67.31))
     (stroke (width 0) (type default))
@@
     (stroke (width 0) (type default))
   )
+  (wire (pts (xy 138.176 52.324) (xy 141.732 52.324))
+    (stroke (width 0) (type default))
+  )
   (wire (pts (xy 81.534 158.75) (xy 81.534 163.83))
     (stroke (width 0) (type default))
@@
     (effects (font (size 1.27 1.27)) (justify left bottom))
   )
-  (text "RX-: Designer can ~{NRST} or UART_RX" (at 326.644 135.382 0)
+  (text "RX-: Designer can ~{NRST} or UART_RX" (at 321.31 135.128 0)
     (effects (font (size 1.27 1.27)) (justify left bottom))
   )
@@
     (effects (font (size 1.27 1.27)) (justify left bottom))
   )
-  (text "RX+: Designer can SWDO or UART_TX" (at 326.39 133.096 0)
+  (text "RX+: Designer can SWDO or UART_TX" (at 321.056 132.842 0)
     (effects (font (size 1.27 1.27)) (justify left bottom))
   )
@@
     (effects (font (size 1.27 1.27)) (justify left bottom))
   )
-  (hierarchical_label "DAM_RX-" (shape input) (at 280.416 205.232 0) (fields_autoplaced)
+  (hierarchical_label "~{NRST}{slash}RXD" (shape input) (at 280.416 205.232 0) (fields_autoplaced)
     (effects (font (size 1.27 1.27)) (justify left))
   )
@@
     (effects (font (size 1.27 1.27)) (justify left))
   )
-  (hierarchical_label "USB_D-" (shape bidirectional) (at 106.172 52.324 180) (fields_autoplaced)
+  (hierarchical_label "USB_D-" (shape bidirectional) (at 98.552 52.324 180) (fields_autoplaced)
     (effects (font (size 1.27 1.27)) (justify right))
   )
@@
     (effects (font (size 1.27 1.27)) (justify right))
   )
-  (hierarchical_label "DAM_RX+" (shape input) (at 280.416 202.692 0) (fields_autoplaced)
+  (hierarchical_label "SWDO{slash}TXD" (shape input) (at 280.416 202.692 0) (fields_autoplaced)
     (effects (font (size 1.27 1.27)) (justify left))
   )
-  (hierarchical_label "USB_D+" (shape bidirectional) (at 134.366 52.324 0) (fields_autoplaced)
+  (hierarchical_label "USB_D+" (shape bidirectional) (at 141.732 52.324 0) (fields_autoplaced)
     (effects (font (size 1.27 1.27)) (justify left))
   )
@@
     (effects (font (size 1.27 1.27)) (justify right))
   )
-  (hierarchical_label "DAM_RX-" (shape input) (at 375.92 134.874 180) (fields_autoplaced)
+  (hierarchical_label "~{NRST}{slash}RXD" (shape input) (at 375.92 134.874 180) (fields_autoplaced)
     (effects (font (size 1.27 1.27)) (justify right))
   )
@@
     (effects (font (size 1.27 1.27)) (justify right))
   )
-  (hierarchical_label "DAM_RX+" (shape input) (at 375.92 132.334 180) (fields_autoplaced)
+  (hierarchical_label "SWDO{slash}TXD" (shape input) (at 375.92 132.334 180) (fields_autoplaced)
     (effects (font (size 1.27 1.27)) (justify right))
   )
@@
     )
   )
+  (symbol (lib_id "Connector:TestPoint_Small") (at 101.6 52.324 0) (unit 1)
+    (in_bom yes) (on_board yes) (dnp no)
+    (property "Reference" "TP9" (at 101.6 50.927 0)
+      (effects (font (size 1.27 1.27)) (justify left))
+    )
+    (property "Value" "TestPoint" (at 103.0732 51.5874 0)
+      (effects (font (size 1.27 1.27)) (justify left) hide)
+    )
+    (property "Footprint" "TestPoint:TestPoint_Pad_D2.0mm" (at 106.68 52.324 0)
+      (effects (font (size 1.27 1.27)) hide)
+    )
+    (property "Datasheet" "~" (at 106.68 52.324 0)
+      (effects (font (size 1.27 1.27)) hide)
+    )
+    (property "Config" "nofit" (at 101.6 52.324 0)
+      (effects (font (size 1.27 1.27)) hide)
+    )
+    (property "MFN" "" (at 101.6 52.324 0)
+      (effects (font (size 1.27 1.27)) hide)
+    )
+    (property "MPN" "" (at 101.6 52.324 0)
+      (effects (font (size 1.27 1.27)) hide)
+    )
+    (property "Description" "" (at 101.6 52.324 0)
+      (effects (font (size 1.27 1.27)) hide)
+    )
+    (property "Notes" "" (at 101.6 52.324 0)
+      (effects (font (size 1.27 1.27)) hide)
+    )
+    (property "Vendor" "" (at 101.6 52.324 0)
+      (effects (font (size 1.27 1.27)) hide)
+    )
+    (property "SKU" "" (at 101.6 52.324 0)
+      (effects (font (size 1.27 1.27)) hide)
+    )
+    (property "Characteristics" "" (at 101.6 52.324 0)
+      (effects (font (size 1.27 1.27)) hide)
+    )
+    (pin "1")
+    (instances
+      (project "USB"
+        (path "/abe08c89-73f7-4625-b1e5-d5b33729a7ca"
+          (reference "TP9") (unit 1)
+        )
+      )
+      (project "spirit_logger_hardware"
+        (path "/e63e39d7-6ac0-4ffd-8aa3-1841a4541b55/cec0ac2b-8788-4205-bc11-fcadefc26e0e"
+          (reference "TP9") (unit 1)
+        )
+      )
+      (project "usb-dam"
+        (path "/eb1f9132-3dcd-4de4-9f05-c2db01d52e0f"
+          (reference "TP1") (unit 1)
+        )
+      )
+    )
+  )
   (symbol (lib_id "power:VCC") (at 196.85 57.658 0) (unit 1)
     (in_bom yes) (on_board yes) (dnp no)
@@
         )
       )
+    )
+  )
+  (symbol (lib_id "Connector:TestPoint_Small") (at 138.176 52.324 0) (unit 1)
+    (in_bom yes) (on_board yes) (dnp no)
+    (property "Reference" "TP9" (at 138.176 50.927 0)
+      (effects (font (size 1.27 1.27)) (justify left))
+    )
+    (property "Value" "TestPoint" (at 139.6492 51.5874 0)
+      (effects (font (size 1.27 1.27)) (justify left) hide)
+    )
+    (property "Footprint" "TestPoint:TestPoint_Pad_D2.0mm" (at 143.256 52.324 0)
+      (effects (font (size 1.27 1.27)) hide)
+    )
+    (property "Datasheet" "~" (at 143.256 52.324 0)
+      (effects (font (size 1.27 1.27)) hide)
+    )
+    (property "Config" "nofit" (at 138.176 52.324 0)
+      (effects (font (size 1.27 1.27)) hide)
+    )
+    (property "MFN" "" (at 138.176 52.324 0)
+      (effects (font (size 1.27 1.27)) hide)
+    )
+    (property "MPN" "" (at 138.176 52.324 0)
+      (effects (font (size 1.27 1.27)) hide)
+    )
+    (property "Description" "" (at 138.176 52.324 0)
+      (effects (font (size 1.27 1.27)) hide)
+    )
+    (property "Notes" "" (at 138.176 52.324 0)
+      (effects (font (size 1.27 1.27)) hide)
+    )
+    (property "Vendor" "" (at 138.176 52.324 0)
+      (effects (font (size 1.27 1.27)) hide)
+    )
+    (property "SKU" "" (at 138.176 52.324 0)
+      (effects (font (size 1.27 1.27)) hide)
+    )
+    (property "Characteristics" "" (at 138.176 52.324 0)
+      (effects (font (size 1.27 1.27)) hide)
+    )
+    (pin "1")
+    (instances
+      (project "USB"
+        (path "/abe08c89-73f7-4625-b1e5-d5b33729a7ca"
+          (reference "TP9") (unit 1)
+        )
+      )
+      (project "spirit_logger_hardware"
+        (path "/e63e39d7-6ac0-4ffd-8aa3-1841a4541b55/cec0ac2b-8788-4205-bc11-fcadefc26e0e"
+          (reference "TP9") (unit 1)
+        )
+      )
+      (project "usb-dam"
+        (path "/eb1f9132-3dcd-4de4-9f05-c2db01d52e0f"
+          (reference "TP6") (unit 1)
+        )
+      )

Commit message: README started
Connections:
- net SWDCLK renamed SWCLK
- net SWDO/TXD renamed SWO/TXD
Other:
- note added: "RX+: Designer can SWO or UART_TX"
- note removed: "RX+: Designer can SWDO or UART_TX"
Changed lines of the file:
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@@
     (title "SWD over DAM (Debug Accessory Mode) Example Board")
     (date "2023-05-16")
-    (rev "0")
+    (rev "1")
     (company "JBR Engineering Research Ltd")
     (comment 1 "J.Whittington 2023")
@@
     (effects (font (size 1.27 1.27)) (justify left bottom))
   )
-  (text "RX+: Designer can SWDO or UART_TX" (at 321.056 132.842 0)
+  (text "RX+: Designer can SWO or UART_TX" (at 321.056 132.842 0)
     (effects (font (size 1.27 1.27)) (justify left bottom))
   )
@@
     (effects (font (size 1.27 1.27)) (justify right))
   )
-  (hierarchical_label "SWDO{slash}TXD" (shape input) (at 280.416 202.692 0) (fields_autoplaced)
+  (hierarchical_label "SWO{slash}TXD" (shape input) (at 280.416 202.692 0) (fields_autoplaced)
     (effects (font (size 1.27 1.27)) (justify left))
   )
@@
     (effects (font (size 1.27 1.27)) (justify left))
   )
-  (hierarchical_label "SWDCLK" (shape input) (at 375.92 129.794 180) (fields_autoplaced)
+  (hierarchical_label "SWCLK" (shape input) (at 375.92 129.794 180) (fields_autoplaced)
     (effects (font (size 1.27 1.27)) (justify right))
   )
@@
     (effects (font (size 1.27 1.27)) (justify left))
   )
-  (hierarchical_label "SWDCLK" (shape input) (at 280.416 200.152 0) (fields_autoplaced)
+  (hierarchical_label "SWCLK" (shape input) (at 280.416 200.152 0) (fields_autoplaced)
     (effects (font (size 1.27 1.27)) (justify left))
   )
@@
     (effects (font (size 1.27 1.27)) (justify right))
   )
-  (hierarchical_label "SWDO{slash}TXD" (shape input) (at 375.92 132.334 180) (fields_autoplaced)
+  (hierarchical_label "SWO{slash}TXD" (shape input) (at 375.92 132.334 180) (fields_autoplaced)
     (effects (font (size 1.27 1.27)) (justify right))
   )

Commit message: pcb render
active layers
Other:
- note added: "RX+: Designer can SWO or UART_TXD"
- note added: "RX-: Designer can ~{NRST} or UART_RXD"
- note removed: "RX+: Designer can SWO or UART_TX"
- note removed: "RX-: Designer can ~{NRST} or UART_RX"
Changed lines of the file:
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@@
     (effects (font (size 1.27 1.27)) (justify left bottom))
   )
-  (text "RX-: Designer can ~{NRST} or UART_RX" (at 321.31 135.128 0)
+  (text "RX-: Designer can ~{NRST} or UART_RXD" (at 321.31 135.128 0)
     (effects (font (size 1.27 1.27)) (justify left bottom))
   )
@@
     (effects (font (size 1.27 1.27)) (justify left bottom))
   )
-  (text "RX+: Designer can SWO or UART_TX" (at 321.056 132.842 0)
+  (text "RX+: Designer can SWO or UART_TXD" (at 321.056 132.842 0)
     (effects (font (size 1.27 1.27)) (justify left bottom))
   )

Commit message: fix example AND footprint VCC 5->6
Connections:
- net VCC: now also U4.6 (VCC); no longer U4.5 (VCC)
Changed lines of the file:
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@@
     (pin "3")
     (pin "4")
-    (pin "5")
+    (pin "6")
     (instances
       (project "usb-dam"
