File: DAMLink.kicad_sch (KiCad schematic)
At the start: 67 parts, among them J1 PicoBlade, J3 PicoBlade, J3 USB_C_Receptacle_Host, J4 VCCIO_EXT, J5 TC2050-IDC, J6 Conn_ST_STDC14, P1 USB_C_Plug, SW1 SW_DIP_x04, U1 FT230XQ, U2 USB3740B-AI2, U3 TMUX1574RSVR, U4 USBLC6-4SC6, U5 SiP32432DR3, U6 USBLC6-4SC6

Commit message: Remove wrong libraries
Remove "altium" libraries which where downloaded wrong from SnapEDA.

Import correct libraries from Manufracturer and from UltranLibrary

Clear whole PCB.
Parts:
- J5: footprint TC2050-IDC:TAG-CONNECT_TC2050-IDC -> Connector:Tag-Connect_TC2050-IDC-FP_2x05_P1.27mm_Vertical
- U3: footprint TMUX1574RSVR:IC_TMUX1574RSVR -> TMUX1574RSVR:RSV16_TEX
Connections:
- net GND: now also J6.5 (GND), J6.7 (GND); no longer J6.05 (GND), J6.07 (GND)
- net SWCLK: now also J6.6 (JCLK/SWCLK); no longer J6.06 (JCLK/SWCLK)
- net SWDIO: now also J6.4 (JTMS/SWDIO); no longer J6.04 (JTMS/SWDIO)
- net SWO: now also J6.8 (JTDO/SWO); no longer J6.08 (JTDO/SWO)
- net VREF: now also J6.3 (VCC); no longer J6.03 (VCC)
Changed lines of the file:
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@@
 			)
 		)
-		(property "Footprint" "TMUX1574RSVR:IC_TMUX1574RSVR"
+		(property "Footprint" "TMUX1574RSVR:RSV16_TEX"
 			(at 320.04 201.93 0)
 			(effects
@@
 			)
 		)
-		(property "Footprint" "TC2050-IDC:TAG-CONNECT_TC2050-IDC"
+		(property "Footprint" "Connector:Tag-Connect_TC2050-IDC-FP_2x05_P1.27mm_Vertical"
 			(at 523.24 157.48 0)
 			(effects
@@
 		(pin "13"
 		)
-		(pin "05"
+		(pin "4"
 		)
-		(pin "07"
+		(pin "7"
 		)
 		(pin "14"
 		)
-		(pin "04"
+		(pin "8"
 		)
 		(pin "10"
 		)
-		(pin "01"
+		(pin "6"
 		)
-		(pin "08"
+		(pin "9"
 		)
-		(pin "03"
+		(pin "2"
 		)
 		(pin "12"
@@
 		(pin "11"
 		)
-		(pin "09"
+		(pin "1"
 		)
-		(pin "06"
+		(pin "3"
 		)
-		(pin "02"
+		(pin "5"
 		)
 		(instances
